Commit message: Cap nhat controller va them thu muc worlds

File: src/spider_controller/urdf/spider.urdf (robot description, URDF)
Before this commit: robot spider, 1 links, 0 joints
Links:
- added link camera_link, mass 0.01; collision box size=0.02 0.05 0.02; visual box size=0.02 0.05 0.02
- added link dummy_link
Joints:
- added joint camera_joint: type fixed, parent base_link, child camera_link, origin xyz=0.15 0 0.05 rpy=0 0 0
- added joint dummy_joint: type fixed, parent dummy_link, child base_link
